Commit message: added pseudo-link to hand tip

File: beo_arm_m4/urdf/beo_arm_m4.urdf (robot description, URDF)
Before this commit: robot beo_arm_m4, 8 links, 7 joints
Links:
- added link hand_tip, mass 0.001; collision box size=0.001 0.001 0.001; visual box size=0.001 0.001 0.001
Joints:
- added joint joint_6: type fixed, parent hand, child hand_tip, origin xyz=0.17 0 0.03 rpy=0 0 0, axis 0 0 0
